File: Eagle/Unbricker.sch (EAGLE design)
At the start: 7 parts, among them J3 M50-3600542, Q1 2N3906

Commit message: Fix power line, add standoffs, etc.
Connections:
- net VCC: now also J2.12; no longer J2.10
Changed lines of the file:
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@@
 <setting verticaltext="up"/>
 </settings>
-<grid distance="0.1" unitdist="inch" unit="inch" style="lines" multiple="1" display="yes" altdistance="0.01" altunitdist="inch" altunit="inch"/>
+<grid distance="0.1" unitdist="inch" unit="inch" style="lines" multiple="1" display="no" altdistance="0.01" altunitdist="inch" altunit="inch"/>
 <layers>
 <layer number="1" name="Top" color="4" fill="1" visible="no" active="no"/>
@@
 <net name="VCC" class="0">
 <segment>
-<pinref part="J2" gate="G$1" pin="10"/>
-<wire x1="208.28" y1="177.8" x2="246.38" y2="177.8" width="0.1524" layer="91"/>
-<wire x1="246.38" y1="177.8" x2="246.38" y2="175.26" width="0.1524" layer="91"/>
+<wire x1="246.38" y1="182.88" x2="246.38" y2="175.26" width="0.1524" layer="91"/>
 <pinref part="Q1" gate="G$1" pin="E"/>
 <label x="220.98" y="177.8" size="1.778" layer="95"/>
+<pinref part="J2" gate="G$1" pin="12"/>
+<wire x1="208.28" y1="182.88" x2="246.38" y2="182.88" width="0.1524" layer="91"/>
 </segment>
 </net>
